Commit message: feat: urdf: add lidar and imu

File: mobile_robot_nodes/description/mobile_robot.urdf.xacro (robot description, xacro)
@@ -93,3 +93,45 @@
     </xacro:inertial_sphere>
   </link>
+  <link name="imu">
+    <visual>
+      <geometry>
+        <box size="${imu_length} ${imu_width} ${imu_height}"/>
+      </geometry>
+      <material name="plastic"/>
+    </visual>
+    <collision>
+      <geometry>
+        <box size="${imu_length} ${imu_width} ${imu_height}"/>
+      </geometry>
+    </collision>
+    <xacro:inertial_box mass="${imu_mass}" x="${imu_length}" y="${imu_width}" z="${imu_height}">
+      <origin xyz="0 0 0" rpy="0 0 0"/>
+    </xacro:inertial_box>
+  </link>
+  <joint name="imu_joint" type="fixed">
+    <parent link="chassis"/>
+    <child link="imu"/>
+    <origin xyz="${chassis_length / 2} 0 ${chassis_height / 2}" rpy="0 0 0"/>
+  </joint>
+  <link name="lidar">
+    <visual>
+      <geometry>
+        <cylinder radius="${lidar_radius}" length="${lidar_height}"/>
+      </geometry>
+      <material name="plastic"/>
+    </visual>
+    <collision>
+      <geometry>
+        <cylinder radius="${lidar_radius}" length="${lidar_height}"/>
+      </geometry>
+    </collision>
+    <xacro:inertial_cylinder mass="${lidar_mass}" length="${lidar_height}" radius="${lidar_radius}">
+      <origin xyz="0 0 0" rpy="0 0 0"/>
+    </xacro:inertial_cylinder>
+  </link>
+  <joint name="lidar_joint" type="fixed">
+    <parent link="chassis"/>
+    <child link="lidar"/>
+    <origin xyz="${chassis_length / 2} 0 ${chassis_height}" rpy="0 0 0"/>
+  </joint>
 </robot>

File: mobile_robot_nodes/description/properties.xacro (robot description, xacro)
@@ -10,3 +10,10 @@
   <xacro:property name="caster_wheel_radius" value="${wheel_radius/2}"/>
   <xacro:property name="caster_wheel_mass" value="0.1"/>
+  <xacro:property name="imu_length" value="0.02"/>
+  <xacro:property name="imu_width" value="0.02"/>
+  <xacro:property name="imu_height" value="0.01"/>
+  <xacro:property name="imu_mass" value="0.01"/>
+  <xacro:property name="lidar_radius" value="0.035"/>
+  <xacro:property name="lidar_height" value="0.04"/>
+  <xacro:property name="lidar_mass" value="0.15"/>
 </robot>

Commit message: fix: urdf: imu position

File: mobile_robot_nodes/description/mobile_robot.urdf.xacro (robot description, xacro)
@@ -112,5 +112,5 @@
     <parent link="chassis"/>
     <child link="imu"/>
-    <origin xyz="${chassis_length / 2} 0 ${chassis_height / 2}" rpy="0 0 0"/>
+    <origin xyz="${0.25 * chassis_length} 0 ${chassis_height / 2}" rpy="0 0 0"/>
   </joint>
   <link name="lidar">

Commit message: fix: update urdf with actual parameters
some of the values where guessed before
actual assembly

.

File: mobile_robot_nodes/description/mobile_robot.urdf.xacro (robot description, xacro)
@@ -32,5 +32,5 @@
     <parent link="base_link"/>
     <child link="left_wheel"/>
-    <origin xyz="0 ${chassis_width/2 + wheel_length/2} 0" rpy="-${pi / 2} 0 0"/>
+    <origin xyz="0 ${chassis_width/2 + wheel_gap + wheel_length/2} 0" rpy="-${pi / 2} 0 0"/>
     <axis xyz="0 0 1"/>
   </joint>
@@ -38,5 +38,5 @@
     <parent link="base_link"/>
     <child link="right_wheel"/>
-    <origin xyz="0 -${chassis_width/2 + wheel_length/2} 0" rpy="${pi / 2} 0 0"/>
+    <origin xyz="0 -${chassis_width/2 + wheel_gap + wheel_length/2} 0" rpy="${pi / 2} 0 0"/>
     <axis xyz="0 0 -1"/>
   </joint>
@@ -134,5 +134,5 @@
     <parent link="chassis"/>
     <child link="lidar"/>
-    <origin xyz="${chassis_length / 2} 0 ${chassis_height}" rpy="0 0 0"/>
+    <origin xyz="${chassis_length / 2} 0 ${chassis_height + lidar_height/2}" rpy="0 0 0"/>
   </joint>
 </robot>

File: mobile_robot_nodes/description/properties.xacro (robot description, xacro)
@@ -1,11 +1,12 @@
 <robot xmlns:xacro="http://www.ros.org/wiki/xacro">
   <!-- robot properties -->
-  <xacro:property name="chassis_length" value="0.15"/>
-  <xacro:property name="chassis_width" value="0.1"/>
-  <xacro:property name="chassis_height" value="0.05"/>
+  <xacro:property name="chassis_length" value="0.20"/>
+  <xacro:property name="chassis_width" value="0.15"/>
+  <xacro:property name="chassis_height" value="0.09"/>
   <xacro:property name="chassis_mass" value="0.5"/>
-  <xacro:property name="wheel_radius" value="0.0325"/>
-  <xacro:property name="wheel_length" value="0.02"/>
+  <xacro:property name="wheel_radius" value="0.0335"/>
+  <xacro:property name="wheel_length" value="0.027"/>
   <xacro:property name="wheel_mass" value="0.1"/>
+  <xacro:property name="wheel_gap" value="0.007"/>
   <xacro:property name="caster_wheel_radius" value="${wheel_radius/2}"/>
   <xacro:property name="caster_wheel_mass" value="0.1"/>
@@ -14,5 +15,5 @@
   <xacro:property name="imu_height" value="0.01"/>
   <xacro:property name="imu_mass" value="0.01"/>
-  <xacro:property name="lidar_radius" value="0.035"/>
+  <xacro:property name="lidar_radius" value="0.04"/>
   <xacro:property name="lidar_height" value="0.04"/>
   <xacro:property name="lidar_mass" value="0.15"/>

File: mobile_robot_nodes/description/ros2_control.xacro (robot description, xacro)
@@ -22,5 +22,5 @@
       <param name="control_rate_hz">200</param>
       <param name="report_rate_hz">50</param>
-      <param name="invert_left">false</param>
+      <param name="invert_left">true</param>
       <param name="invert_right">false</param>
     </hardware>

Commit message: feat(nodes): add use_mock_hardware, use_lidar and use_foxglove launch args
use_mock_hardware:=true swaps MobileRobotHardware for
mock_components/GenericSystem (calculate_dynamics, so odometry moves).
use_lidar/use_foxglove gate the xv_11 driver and foxglove_bridge.
Defaults keep the robot's behavior.

File: mobile_robot_nodes/description/mobile_robot.urdf.xacro (robot description, xacro)
@@ -1,3 +1,5 @@
 <robot xmlns:xacro="http://www.ros.org/wiki/xacro" name="mobile_robot">
+  <!-- true: mock_components/GenericSystem instead of the esp32, see ros2_control.xacro -->
+  <xacro:arg name="use_mock_hardware" default="false"/>
   <xacro:include filename="properties.xacro"/>
   <xacro:include filename="materials.xacro"/>

File: mobile_robot_nodes/description/ros2_control.xacro (robot description, xacro)
@@ -1,27 +1,39 @@
 <robot xmlns:xacro="http://www.ros.org/wiki/xacro">
+  <!-- use_mock_hardware:=true swaps the esp32 for mock_components/GenericSystem
+       so the stack runs on a dev machine / in tests without hardware -->
+  <xacro:arg name="use_mock_hardware" default="false"/>
+  <xacro:property name="use_mock_hardware" value="$(arg use_mock_hardware)"/>
   <ros2_control name="mobile_robot_ros2_control" type="system">
     <hardware>
-      <plugin>mobile_robot_hardware/MobileRobotHardware</plugin>
-      <!-- list all params here that are needed by the hardware plugin - it will receive them  -->
-      <!-- through the info object. e.g. baud_rate, serial_port ... -->
-      <param name="serial_port">/dev/esp32</param>
-      <param name="baud_rate">115200</param>
-      <!-- PI gains, shared by both wheels, integral limit is a duty fraction -->
-      <param name="pid_kp">0.5</param>
-      <param name="pid_ki">2.0</param>
-      <param name="pid_integral_limit">0.3</param>
-      <!-- feedforward per wheel, slope in duty fraction per (rad/s),
-           min_duty in [0,1) compensates the motor deadband -->
-      <param name="ff_slope_left">0.1</param>
-      <param name="ff_slope_right">0.1</param>
-      <param name="ff_min_duty_left">0.0</param>
-      <param name="ff_min_duty_right">0.0</param>
-      <param name="ticks_per_wheel_rev">480</param>
-      <!-- report_rate_hz must not exceed control_rate_hz -->
-      <param name="watchdog_timeout_ms">200</param>
-      <param name="control_rate_hz">200</param>
-      <param name="report_rate_hz">50</param>
-      <param name="invert_left">true</param>
-      <param name="invert_right">false</param>
+      <xacro:if value="${use_mock_hardware}">
+        <plugin>mock_components/GenericSystem</plugin>
+        <!-- integrate the commanded velocity into the position state, so
+             odometry moves like on the real robot -->
+        <param name="calculate_dynamics">true</param>
+      </xacro:if>
+      <xacro:unless value="${use_mock_hardware}">
+        <plugin>mobile_robot_hardware/MobileRobotHardware</plugin>
+        <!-- list all params here that are needed by the hardware plugin - it will receive them  -->
+        <!-- through the info object. e.g. baud_rate, serial_port ... -->
+        <param name="serial_port">/dev/esp32</param>
+        <param name="baud_rate">115200</param>
+        <!-- PI gains, shared by both wheels, integral limit is a duty fraction -->
+        <param name="pid_kp">0.5</param>
+        <param name="pid_ki">2.0</param>
+        <param name="pid_integral_limit">0.3</param>
+        <!-- feedforward per wheel, slope in duty fraction per (rad/s),
+             min_duty in [0,1) compensates the motor deadband -->
+        <param name="ff_slope_left">0.1</param>
+        <param name="ff_slope_right">0.1</param>
+        <param name="ff_min_duty_left">0.0</param>
+        <param name="ff_min_duty_right">0.0</param>
+        <param name="ticks_per_wheel_rev">480</param>
+        <!-- report_rate_hz must not exceed control_rate_hz -->
+        <param name="watchdog_timeout_ms">200</param>
+        <param name="control_rate_hz">200</param>
+        <param name="report_rate_hz">50</param>
+        <param name="invert_left">true</param>
+        <param name="invert_right">false</param>
+      </xacro:unless>
     </hardware>
     <joint name="left_wheel_joint">
@@ -30,6 +42,14 @@
         <param name="max" value="10.0"/>
       </command_interface>
-      <state_interface name="velocity"/>
-      <state_interface name="position"/>
+      <state_interface name="velocity">
+        <xacro:if value="${use_mock_hardware}">
+          <param name="initial_value">0.0</param>
+        </xacro:if>
+      </state_interface>
+      <state_interface name="position">
+        <xacro:if value="${use_mock_hardware}">
+          <param name="initial_value">0.0</param>
+        </xacro:if>
+      </state_interface>
     </joint>
     <joint name="right_wheel_joint">
@@ -38,6 +58,14 @@
         <param name="max" value="10.0"/>
       </command_interface>
-      <state_interface name="velocity"/>
-      <state_interface name="position"/>
+      <state_interface name="velocity">
+        <xacro:if value="${use_mock_hardware}">
+          <param name="initial_value">0.0</param>
+        </xacro:if>
+      </state_interface>
+      <state_interface name="position">
+        <xacro:if value="${use_mock_hardware}">
+          <param name="initial_value">0.0</param>
+        </xacro:if>
+      </state_interface>
     </joint>
   </ros2_control>
